Commit message: Add ros_planar_move_plugin to timda_mobile_platform.urdf.xacro

File: wrs_gazebo/timda_mobile_platform/urdf/timda_mobile_platform.urdf.xacro (robot description, xacro)
@@ -3,5 +3,23 @@
      Commit Version: 1.5.1-0-g916b5db  Build Version: 1.5.7152.31018
      For more information, please see http://wiki.ros.org/sw_urdf_exporter -->
-<robot name="timda_mobile_platform">
+<robot xmlns:xacro="http://www.ros.org/wiki/xacro" name="timda_mobile_platform">
+  <gazebo>
+    <plugin name="object_controller" filename="libgazebo_ros_planar_move.so">
+      <commandTopic>cmd_vel</commandTopic>
+      <odometryTopic>odom</odometryTopic>
+      <odometryFrame>odom</odometryFrame>
+      <odometryRate>20.0</odometryRate>
+      <robotBaseFrame>base_footprint</robotBaseFrame>
+    </plugin>
+  </gazebo>
+  <gazebo reference="base_link">
+    <material>Gazebo/DarkGrey</material>
+  </gazebo>
+  <link name="base_footprint"/>
+  <joint name="base_link_joint" type="fixed">
+    <origin xyz="0.0 0 0.01" rpy="0 0 0" />
+    <parent link="base_footprint"/>
+    <child link="base_link" />
+  </joint>
   <link name="base_link">
     <inertial>

Commit message: Seperate gazebo plugin from urdf.xacro

File: wrs_gazebo/timda_mobile_platform/urdf/timda_mobile_platform.urdf.xacro (robot description, xacro)
@@ -4,16 +4,5 @@
      For more information, please see http://wiki.ros.org/sw_urdf_exporter -->
 <robot xmlns:xacro="http://www.ros.org/wiki/xacro" name="timda_mobile_platform">
-  <gazebo>
-    <plugin name="object_controller" filename="libgazebo_ros_planar_move.so">
-      <commandTopic>cmd_vel</commandTopic>
-      <odometryTopic>odom</odometryTopic>
-      <odometryFrame>odom</odometryFrame>
-      <odometryRate>20.0</odometryRate>
-      <robotBaseFrame>base_footprint</robotBaseFrame>
-    </plugin>
-  </gazebo>
-  <gazebo reference="base_link">
-    <material>Gazebo/DarkGrey</material>
-  </gazebo>
+  <xacro:include filename="$(find timda_mobile_platform)/urdf/timda_mobile_platform.gazebo.xacro" />
   <link name="base_footprint"/>
   <joint name="base_link_joint" type="fixed">
